File: wall/wall.sch (KiCad schematic (older format))
At the start: 83 parts, among them J1 CON

Commit message: finished wall
Parts:
- added C42, C43: 100n, otter:C_0402, symbol Device:C_Small
- added J2: Conn_01x02, otter:conn_01x02_smd_2mm, symbol Connector_Generic:Conn_01x02
Connections:
- net DOUT: now also D41.4 (DOUT)
- net GND: now also C42.1, C42.2, C43.1, C43.2, J2.1 (Pin_1), J2.2 (Pin_2)
Changed lines of the file:
@@
 Wire Wire Line
 	4700 1200 4950 1200
+Text GLabel 10900 6200 2    50   Input ~ 0
+DOUT
+$Comp
+L otter:GND #PWR0152
+U 1 1 61F8E1B5
+P 2200 4400
+F 0 "#PWR0152" H 2200 4150 50  0001 C CNN
+F 1 "GND" V 2205 4272 50  0000 R CNN
+F 2 "" H 2200 4400 60  0000 C CNN
+F 3 "" H 2200 4400 60  0000 C CNN
+	1    2200 4400
+	0    1    1    0
+$EndComp
+$Comp
+L Connector_Generic:Conn_01x02 J2
+U 1 1 61FB2B8A
+P 2400 4350
+F 0 "J2" H 2480 4342 50  0000 L CNN
+F 1 "Conn_01x02" H 2480 4251 50  0000 L CNN
+F 2 "otter:conn_01x02_smd_2mm" H 2400 4350 50  0001 C CNN
+F 3 "~" H 2400 4350 50  0001 C CNN
+	1    2400 4350
+	1    0    0    -1
+$EndComp
+Wire Wire Line
+	2200 4350 2200 4400
+Connection ~ 2200 4400
+Wire Wire Line
+	2200 4400 2200 4450
+$Comp
+L Device:C_Small C42
+U 1 1 61FC0E05
+P 2400 5050
+F 0 "C42" V 2629 5050 50  0000 C CNN
+F 1 "100n" V 2538 5050 50  0000 C CNN
+F 2 "otter:C_0402" H 2400 5050 50  0001 C CNN
+F 3 "~" H 2400 5050 50  0001 C CNN
+	1    2400 5050
+	0    -1   -1   0
+$EndComp
+$Comp
+L otter:GND #PWR0153
+U 1 1 61FC0E0B
+P 2500 5050
+F 0 "#PWR0153" H 2500 4800 50  0001 C CNN
+F 1 "GND" V 2505 4922 50  0000 R CNN
+F 2 "" H 2500 5050 60  0000 C CNN
+F 3 "" H 2500 5050 60  0000 C CNN
+	1    2500 5050
+	0    -1   -1   0
+$EndComp
+$Comp
+L otter:GND #PWR0154
+U 1 1 61FC983F
+P 2300 5050
+F 0 "#PWR0154" H 2300 4800 50  0001 C CNN
+F 1 "GND" V 2305 4922 50  0000 R CNN
+F 2 "" H 2300 5050 60  0000 C CNN
+F 3 "" H 2300 5050 60  0000 C CNN
+	1    2300 5050
+	0    1    1    0
+$EndComp
+$Comp
+L Device:C_Small C43
+U 1 1 61FD4D3F
+P 2400 5400
+F 0 "C43" V 2629 5400 50  0000 C CNN
+F 1 "100n" V 2538 5400 50  0000 C CNN
+F 2 "otter:C_0402" H 2400 5400 50  0001 C CNN
+F 3 "~" H 2400 5400 50  0001 C CNN
+	1    2400 5400
+	0    -1   -1   0
+$EndComp
+$Comp
+L otter:GND #PWR0155
+U 1 1 61FD4D45
+P 2500 5400
+F 0 "#PWR0155" H 2500 5150 50  0001 C CNN
+F 1 "GND" V 2505 5272 50  0000 R CNN
+F 2 "" H 2500 5400 60  0000 C CNN
+F 3 "" H 2500 5400 60  0000 C CNN
+	1    2500 5400
+	0    -1   -1   0
+$EndComp
+$Comp
+L otter:GND #PWR0156
+U 1 1 61FD4D4B
+P 2300 5400
+F 0 "#PWR0156" H 2300 5150 50  0001 C CNN
+F 1 "GND" V 2305 5272 50  0000 R CNN
+F 2 "" H 2300 5400 60  0000 C CNN
+F 3 "" H 2300 5400 60  0000 C CNN
+	1    2300 5400
+	0    1    1    0
+$EndComp
 $EndSCHEMATC
