File: wall/wall.kicad_pcb (KiCad board)
At the start: 2 copper layers, 40 x 180 mm, 83 parts, among them J1 CON

Commit message: finished wall
Parts:
- added C42: 100n, otter:C_0402, B.Cu at (134.5, 22.1)
- added C43: 100n, otter:C_0402, B.Cu at (113.7, 22.1)
- added G***: LOGO, otter:laemp_wall-text, B.Cu at (120.0, 198.2)
- added J2: Conn_01x02, otter:conn_01x02_smd_2mm, B.Cu at (127.2, 27.5)
- moved C13 8.54 mm to (135.8, 101.9), turned to 0 degrees
- moved C37 1.80 mm to (115.5, 159.0)
- moved C41 0.22 mm to (116.3, 123.2)
- moved C34 0.14 mm to (109.5, 87.7)
- moved D22 0.14 mm to (113.7, 86.8)
- moved C11 0.10 mm to (137.3, 61.2)
- moved D35 0.10 mm to (104.3, 53.0)
- turned C32 to 90 degrees
- turned D17 to 270 degrees
Connections:
- D41 pad 4: Net-(D41-Pad4) -> DOUT
Routing:
- net VBUS: track 0.00 -> 708.8 mm
- net DOUT: track 0.00 -> 185.0 mm
- net Net-(D24-Pad4): track 0.00 -> 38.8 mm
- net Net-(D35-Pad4): track 0.00 -> 29.3 mm
- net Net-(D5-Pad4): track 0.00 -> 28.8 mm
- net Net-(D14-Pad4): track 0.00 -> 27.7 mm
- net Net-(D31-Pad4): track 0.00 -> 26.2 mm
- net Net-(D11-Pad4): track 0.00 -> 24.8 mm
- net Net-(D19-Pad4): track 0.00 -> 23.5 mm
- net Net-(D32-Pad4): track 0.00 -> 23.5 mm
- net Net-(D16-Pad4): track 0.00 -> 23.2 mm
- net Net-(D23-Pad4): track 0.00 -> 19.8 mm
- net Net-(D22-Pad4): track 0.00 -> 19.2 mm
- net Net-(D1-Pad4): track 0.00 -> 19.2 mm
- net Net-(D25-Pad4): track 0.00 -> 18.9 mm
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- added copper zone on B.Cu, net GND
- added copper zone on F.Cu, net GND
Other:
- net class Default: clearance 0.2 -> 0.127; trace_width 0.25 -> 0.2
- rule pad_to_mask_clearance: 0.051 -> 0
- rule trace_clearance: 0.2 -> 0.127
- board text removed: "particular pinnipeds prefer"

Commit message: finished wall board
Parts:
- moved C42 0.10 mm to (134.5, 22.0)
- moved C43 0.10 mm to (113.7, 22.0)
Other:
- board text added: "LÄMP"
- board text added: "LÄMP wall-board v1.0 by Jana Marie Hemsing @_Jana_Marie 2021 github.com/Jana-Marie/laemp"
Changed lines of the file:
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@@
   (general
     (thickness 1.6)
-    (drawings 33)
+    (drawings 35)
     (tracks 648)
     (zones 0)
@@
   )
   (module otter:C_0402 (layer B.Cu)
-    (at 113.72 22.1)
+    (at 113.72 22)
     (descr "Capacitor 0402")
     (tags "C Capacitor 0402")
@@
   )
   (module otter:C_0402 (layer B.Cu)
-    (at 134.5 22.1)
+    (at 134.5 22)
     (descr "Capacitor 0402")
     (tags "C Capacitor 0402")
@@
     )
   )
-  (gr_text JLCJLCJLCJLC (at 120 187) (layer B.SilkS)
-    (effects (font (size 1 1) (thickness 0.15)) (justify mirror))
+  (gr_text JLCJLCJLCJLC (at 120 186.9) (layer B.SilkS)
+    (effects (font (size 0.8 0.8) (thickness 0.1)) (justify mirror))
+  )
+  (gr_text LÄMP (at 107.4 191.6) (layer B.SilkS)
+    (effects (font (size 3 3) (thickness 0.3)) (justify mirror))
+  )
+  (gr_text "LÄMP wall-board v1.0\nby Jana Marie Hemsing\n@_Jana_Marie 2021\ngithub.com/Jana-Marie/laemp" (at 131.4 191.6) (layer B.SilkS)
+    (effects (font (size 0.65 0.65) (thickness 0.1)) (justify mirror))
   )
   (gr_circle (center 135.25 166.25) (end 137 166.5) (layer Edge.Cuts) (width 0.15))
