File: hex_top/hex_top.kicad_pcb (KiCad board)
At the start: 2 copper layers, 69.3 x 80 mm, 0 parts

Commit message: finished top
Parts:
- added REF**: pad_1.5_3, otter:pad_1.5_3, B.Cu at (89.3, 69.0)
- added REF**: pad_1.5_3, otter:pad_1.5_3, B.Cu at (96.0, 134.9)
- added REF**: pad_1.5_3, otter:pad_1.5_3, B.Cu at (67.8, 93.7)
- added REF**: pad_1.5_3, otter:pad_1.5_3, B.Cu at (67.8, 114.0)
- added REF**: pad_1.5_3, otter:pad_1.5_3, B.Cu at (71.8, 79.1)
- added REF**: pad_1.5_3, otter:pad_1.5_3, B.Cu at (121.5, 75.3)
- added REF**: pad_1.5_3, otter:pad_1.5_3, B.Cu at (104.0, 65.1)
- added REF**: pad_1.5_3, otter:pad_1.5_3, B.Cu at (132.2, 106.3)
- added REF**: pad_1.5_3, otter:pad_1.5_3, B.Cu at (132.2, 86.0)
- added REF**: pad_1.5_3, otter:pad_1.5_3, B.Cu at (110.7, 131.0)
- added REF**: pad_1.5_3, otter:pad_1.5_3, B.Cu at (128.2, 120.9)
- added REF**: pad_1.5_3, otter:pad_1.5_3, B.Cu at (78.5, 124.7)
Other:
- outline, holes or cut-outs redrawn
