File: hex_led_board/hex_led_board.kicad_pcb (KiCad board)
At the start: 2 copper layers, 69.3 x 80 mm, 90 parts, among them J1 Conn_01x04, J2 Conn_01x04

Commit message: updated files
Other:
- net class Default removed
