File: hex_base/hex_base.kicad_sch (KiCad schematic)
At the start: 47 parts

Commit message: updated file
Parts:
- added D2: D_Small, Diode_SMD:D_SOD-123F, symbol Device:D_Small
- added R16: DNP, otter:R_0402, symbol Device:R_Small
- added R17: 20, otter:R_0402, symbol Device:R_Small
- C1, C11, C12, C2, C3, C5, C6, C9: value (none) -> 100n; footprint (none) -> otter:C_0402
- C10, C4, C7, C8: value (none) -> 10u; footprint (none) -> otter:C_0603
- D1: value (none) -> SK6812; footprint (none) -> LED_SMD:LED_SK6812_PLCC4_5.0x5.0mm_P3.2mm
- J1: value (none) -> ESP_proc; footprint (none) -> Connector_PinHeader_2.54mm:PinHeader_1x05_P2.54mm_Vertical
- J10: value (none) -> PANEL5; footprint (none) -> otter:PinSocket_1x06_P2.00mm_Vertical_center
- J11: value (none) -> LED_HEX0; footprint (none) -> otter:PinSocket_1x04_P2.54mm_Vertical_center
- J12: value (none) -> LED_HEX1; footprint (none) -> otter:PinSocket_1x04_P2.54mm_Vertical_center
- J2: value (none) -> E75_proc; footprint (none) -> Connector_PinHeader_2.54mm:PinHeader_1x05_P2.54mm_Vertical
- J3: value (none) -> USB_C; footprint (none) -> otter:USB-C 16Pin; symbol hex_base-rescue:USB_C_Receptacle_USB2.0-Connector -> Connector:USB_C_Receptacle_USB2.0
- J4, J5: value (none) -> PANEL0; footprint (none) -> otter:PinSocket_1x03_P2.00mm_Vertical
- J6: value (none) -> PANEL1; footprint (none) -> otter:PinSocket_1x06_P2.00mm_Vertical_center
- J7: value (none) -> PANEL2; footprint (none) -> otter:PinSocket_1x06_P2.00mm_Vertical_center
- J8: value (none) -> PANEL3; footprint (none) -> otter:PinSocket_1x06_P2.00mm_Vertical_center
- J9: value (none) -> PANEL4; footprint (none) -> otter:PinSocket_1x06_P2.00mm_Vertical_center
- P1: value (none) -> TC2030-ESP; footprint (none) -> otter:TC2030
- P2: value (none) -> TC2030-E75; footprint (none) -> otter:TC2030
- R1: value (none) -> R_PHOTO; footprint (none) -> otter:R_0805; symbol hex_base-rescue:R_PHOTO-Device -> Device:R_PHOTO
- R10, R11, R12, R15, R2, R8: value (none) -> 100k; footprint (none) -> otter:R_0402
- R13, R14, R3, R4, R5, R6, R7: value (none) -> 5k1; footprint (none) -> otter:R_0402
- R9: value (none) -> 20; footprint (none) -> otter:R_0402
- SW1: value (none) -> RST; footprint (none) -> Button_Switch_SMD:SW_SPST_PTS810
- SW2: value (none) -> BIND; footprint (none) -> Button_Switch_SMD:SW_SPST_PTS810
- U1: value (none) -> ESP32-WROOM-32; footprint (none) -> RF_Module:ESP32-WROOM-32
- U2: value (none) -> E75-2G4M20S; footprint (none) -> otter:E75-2G4M10S
- U3: value (none) -> AMS1117-3.3; footprint (none) -> Package_TO_SOT_SMD:SOT-223-3_TabPin2
Connections:
- net DOUT: now also R16.1
- net SK6812: now also R17.1; no longer D1.4 (DOUT)
- net VBUS: now also D2.2 (A); no longer C6.2, D1.3 (VDD)
- new net: C6.2, D1.3 (VDD), D2.1 (K)
- new net: D1.4 (DOUT), R16.2, R17.2
Other:
- moved on the sheet: C6, D1, R8, R9
